File: openffboard-esp32s2/esp32s2-openffb.kicad_pcb (KiCad board)
At the start: 2 copper layers, 60 x 60 mm, 54 parts, among them J1 USB_C_Receptacle_USB2.0, J2 Debug, J3 CAN_Connector, J4 Motor Driver, J5 INPUTS, J6 ENCODER & PWM, SW1 SW_Push, SW2 SW_Push, U1 AMS1117-3.3, U2 ESP32-S2FH4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

Commit message: v1.1
Parts:
- removed AE1: Antenna_Chip, RF_Antenna:Johanson_2450AT43F0100
- removed C10, C16, C17, C8: TBD, Capacitor_SMD:C_0402_1005Metric
- removed C11, C12, C13, C14, C3, C5, C7, C9: 0.1uf, Capacitor_SMD:C_0402_1005Metric
- removed D2: ESD9B3.3ST5G, Diode_SMD:D_SOD-923
- removed L1: L, Inductor_SMD:L_0402_1005Metric
- removed L2: 2nH, Inductor_SMD:L_0402_1005Metric
- removed REF**: OSHW-Logo2_9.8x8mm_SilkScreen, Symbol:OSHW-Logo2_9.8x8mm_SilkScreen
- removed U2: ESP32-S2FH4, Package_DFN_QFN:QFN-56-1EP_7x7mm_P0.4mm_EP5.6x5.6mm
- removed Y1: 40MHz(±10ppm), Crystal:Crystal_SMD_EuroQuartz_MT-4Pin_3.2x2.5mm
- added C19: 10uf, Capacitor_SMD:C_0603_1608Metric, F.Cu at (137.0, 67.7)
- added J7: RJ12, Connector_RJ:RJ25_Wayconn_MJEA-660X1_Horizontal, F.Cu at (144.7, 65.3)
- added R10: 5.1k, Resistor_SMD:R_0402_1005Metric, F.Cu at (135.9, 64.4)
- added R11: 5.1k, Resistor_SMD:R_0402_1005Metric, F.Cu at (131.3, 64.4)
- added R12: 5.1k, Resistor_SMD:R_0402_1005Metric, F.Cu at (164.3, 72.6)
- added R13: 5.1k, Resistor_SMD:R_0402_1005Metric, F.Cu at (167.2, 70.7)
- added U4: USBLC6-2SC6, Package_TO_SOT_SMD:SOT-23-6, F.Cu at (133.6, 65.3)
- added U5: ESP32-S2-SOLO, Espressif:ESP32-S2-SOLO, F.Cu at (163.6, 87.3)
- added logo1: logo, Symbol:OSHW-Logo2_9.8x8mm_SilkScreen, F.Cu at (180.3, 128.4)
- C2: value 4.7uf -> 10uf
- D1: value ESD9B3.3ST5G -> SMAJ5.0CA_400W_5V; footprint Diode_SMD:D_SOD-923 -> Diode_SMD:D_SMA
- J5: value INPUTS -> ENCODER & PWM
- J6: value ENCODER & PWM -> RJ12; footprint Connector_PinHeader_2.54mm:PinHeader_2x05_P2.54mm_Vertical -> Connector_RJ:RJ25_Wayconn_MJEA-660X1_Horizontal
- R5: value 10k -> 5.1k
- moved J1 51.3 mm to (133.8, 58.6), turned to 180 degrees
- moved F1 39.5 mm to (137.9, 65.0), turned to 90 degrees
- moved D1 34.1 mm to (135.4, 70.2), turned to 180 degrees
- moved C1 33.9 mm to (144.9, 77.5), turned to 90 degrees
- moved R1 33.4 mm to (142.9, 70.5), turned to 180 degrees
- moved R2 32.2 mm to (142.9, 71.4), turned to 180 degrees
- moved U1 31.9 mm to (139.7, 79.2), turned to 180 degrees
- moved C2 27.2 mm to (144.9, 80.8), turned to 90 degrees
- moved R5 26.0 mm to (164.3, 70.7)
- moved C15 22.1 mm to (171.1, 76.3), turned to 0 degrees
- moved C4 22.1 mm to (171.6, 75.1)
- moved J2 21.9 mm to (168.0, 111.7), turned to 270 degrees
- moved D12 20.8 mm to (168.6, 106.5), turned to 90 degrees
- moved R6 20.5 mm to (168.7, 103.1), turned to 90 degrees
- moved R7 19.2 mm to (167.7, 103.1), turned to 90 degrees
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Connections:
- D1 pad 1: GND -> +5V
- D1 pad 2: Net-(D1-Pad2) -> GND
- J1 pad A6: Net-(D2-Pad1) -> Net-(J1-PadA6)
- J1 pad A7: Net-(D1-Pad2) -> Net-(J1-PadA7)
- J1 pad A8: Net-(J1-PadA8) -> (no net)
- J1 pad B6: Net-(D2-Pad1) -> Net-(J1-PadA6)
- J1 pad B7: Net-(D1-Pad2) -> Net-(J1-PadA7)
- J1 pad B8: Net-(J1-PadB8) -> (no net)
- J4 pad 13: /V_EXT -> (no net)
- J4 pad 14: /V_INT -> (no net)
- J5 pad 1: /DIN0 -> /ENCODER_A
- J5 pad 10: GND -> +3V3
- J5 pad 2: /AIN0 -> /PWM1
- J5 pad 3: /DIN1 -> /ENCODER_B
- J5 pad 4: /AIN1 -> /PWM2
- J5 pad 5: /DIN2 -> /ENCODER_Z
- J5 pad 6: /AIN2 -> /PWM3
- J5 pad 7: +3V3 -> GND
- J5 pad 8: +3V3 -> /PWM4
- J5 pad 9: GND -> +5V
- J6 pad 1: /ENCODER_A -> GND
- J6 pad 2: /PWM1 -> GND
- J6 pad 3: /ENCODER_B -> +3V3
- J6 pad 4: /PWM2 -> /AIN0
- J6 pad 5: /ENCODER_Z -> /AIN1
- J6 pad 6: /PWM3 -> /AIN2
- R1 pad 1: /USB_D- -> Net-(R1-Pad1)
- R1 pad 2: Net-(D1-Pad2) -> /USB_D-
- R2 pad 1: /USB_D+ -> Net-(R2-Pad1)
- R2 pad 2: Net-(D2-Pad1) -> /USB_D+
- R5 pad 2: Net-(R5-Pad2) -> /AIN2
- SW1 pad 1: Net-(SW1-Pad1) -> /DBG_IO0
Routing:
- net +3V3: track 239.7 -> 0.00 mm, vias 10 -> 0
- net +5V: track 107.6 -> 0.00 mm, vias 2 -> 0
- net /DBG_EN: track 75.4 -> 0.00 mm, vias 6 -> 0
- net /DIN1: track 34.0 -> 0.00 mm, vias 2 -> 0
- net /AIN2: track 33.9 -> 0.00 mm
- net /DIN0: track 31.1 -> 0.00 mm, vias 2 -> 0
- net /AIN1: track 30.9 -> 0.00 mm
- net /DIN2: track 30.7 -> 0.00 mm, vias 2 -> 0
- net /SPI1_MISO: track 29.3 -> 0.00 mm, vias 2 -> 0
- net /SPI1_MOSI: track 26.2 -> 0.00 mm, vias 2 -> 0
- net /DRV_ENABLE: track 26.1 -> 0.00 mm
- net /AIN0: track 25.8 -> 0.00 mm
- net /USB_D-: track 25.5 -> 0.00 mm
- net /ENCODER_A: track 25.4 -> 0.00 mm
- net /ENCODER_B: track 25.0 -> 0.00 mm
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- removed copper zone on F.Cu, net GND
Other:
- outline, holes or cut-outs redrawn
- board text added: "V1.1"
- board text removed: "V1.0"

Commit message: v1.1
Parts:
- removed C18: 10uf, Capacitor_SMD:C_0603_1608Metric
- removed R3: 120Ω, Resistor_SMD:R_0603_1608Metric
- added C3: 10uf, Capacitor_SMD:C_0603_1608Metric, F.Cu at (145.5, 97.9)
- added R15: 120Ω, Resistor_SMD:R_0603_1608Metric, F.Cu at (135.9, 97.9)
- added U2: ESP32-S3-WROOM-1, Espressif:ESP32-S3-WROOM-1, F.Cu at (163.6, 87.3)
- moved logo1 52.5 mm to (133.0, 105.8)
- moved J2 20.4 mm to (147.6, 111.6)
- moved R2 7.66 mm to (136.4, 67.4)
- moved R1 6.85 mm to (136.4, 68.3)
- moved D1 6.48 mm to (140.7, 73.9)
- moved R9 4.22 mm to (164.9, 107.2)
- moved D10 4.22 mm to (164.6, 110.6)
- moved D11 4.22 mm to (163.1, 110.6)
- moved D12 4.22 mm to (167.6, 110.6)
- moved D9 4.22 mm to (166.1, 110.6)
- moved R6 4.22 mm to (167.7, 107.2)
- moved R7 4.22 mm to (166.8, 107.2)
- moved R8 4.22 mm to (165.8, 107.2)
- moved J3 3.54 mm to (122.3, 102.8), turned to 90 degrees
- moved R13 3.37 mm to (164.0, 69.7), turned to 90 degrees
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Connections:
- J3 pad 1: Net-(J3-Pad1) -> /connector/CANL
- J3 pad 2: Net-(J3-Pad2) -> /connector/CANH
- R1 pad 1: Net-(R1-Pad1) -> /USB_D+
- R1 pad 2: /USB_D- -> /connector/USB_D+
- R2 pad 1: Net-(R2-Pad1) -> /USB_D-
- R2 pad 2: /USB_D+ -> /connector/USB_D-
- U3 pad 6: Net-(J3-Pad2) -> /connector/CANL
- U3 pad 7: Net-(J3-Pad1) -> /connector/CANH
- U4 pad 4: /USB_D+ -> /connector/USB_D+
- U4 pad 6: /USB_D- -> /connector/USB_D-
- U5 pad 10: /SPI1_CS1 -> /PWM4
- U5 pad 12: /ENCODER_Z -> /DIN3
- U5 pad 13: Net-(R1-Pad1) -> /USB_D-
- U5 pad 14: Net-(R2-Pad1) -> /USB_D+
- U5 pad 16: /DIN2 -> /SPI1_SCK
- U5 pad 17: /PWM3 -> /DIN2
- U5 pad 18: /PWM4 -> /DIN1
- U5 pad 19: /GPIO_DRV -> /DIN0
- U5 pad 20: /DRV_ENABLE -> /GPIO_DRV
- U5 pad 21: /DRV_FLAG -> /DRV_ENABLE
- U5 pad 22: /BRAKE_CTRL -> /DRV_FLAG
- U5 pad 23: /SPI1_SCK -> /BRAKE_CTRL
- U5 pad 24: /SPI1_MOSI -> /SPI1_CS2
- U5 pad 25: /SPI1_MISO -> /SPI1_CS3
- U5 pad 26: /DIN0 -> /SPI1_CS1
- U5 pad 31: /DIN3 -> /SPI1_MISO
- U5 pad 32: /LED_ERR -> /SPI1_MOSI
- U5 pad 33: /LED_CLIP -> /LED_ERR
- U5 pad 34: /LED_SYS -> /LED_CLIP
- U5 pad 35: /DIN1 -> /LED_SYS
- U5 pad 8: /SPI1_CS2 -> /ENCODER_Z
- U5 pad 9: /SPI1_CS3 -> /PWM3
Routing:
- net +3V3: track 0.00 -> 221.5 mm, vias 0 -> 6
- net /DBG_EN: track 0.00 -> 108.8 mm, vias 0 -> 5
- net +5V: track 0.00 -> 101.6 mm, vias 0 -> 4
- net /SPI1_SCK: track 0.00 -> 43.5 mm, vias 0 -> 2
- net /DBG_TX: track 0.00 -> 42.6 mm
- net /SPI1_MISO: track 0.00 -> 42.6 mm, vias 0 -> 2
- net /SPI1_MOSI: track 0.00 -> 41.5 mm, vias 0 -> 2
- net /DBG_RX: track 0.00 -> 39.6 mm
- net /AIN0: track 0.00 -> 36.7 mm, vias 0 -> 2
- net /DRV_ENABLE: track 0.00 -> 36.0 mm
- net /BRAKE_CTRL: track 0.00 -> 35.0 mm
- net /SPI1_CS3: track 0.00 -> 35.0 mm
- net /AIN1: track 0.00 -> 33.5 mm, vias 0 -> 2
- net /GPIO_DRV: track 0.00 -> 33.1 mm
- net /DRV_FLAG: track 0.00 -> 31.9 mm
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- added copper zone on F.Cu, net GND
Other:
- board text added: "5V|3V3"
- board text added: "A|PWM1"
- board text added: "B|PWM2"
- board text added: "CS1|SCK"
- board text added: "CS2|CS3"
- board text added: "DRV_GP|EN"
- board text added: "FLAG|BRAKE"
- board text added: "GND|5V"
- board text added: "GND|PWM4"
- board text added: "MOSI|MISO"
- board text added: "RST|3V3"
- board text added: "V_EXT|V_INT"
- board text added: "Z|PWM3"
- board text removed: "3V3|3V3"
- board text removed: "3V3|5V"
- board text removed: "3V3|RST"
- board text removed: "5V|GND"
- board text removed: "BRAKE|FLAG"
- board text removed: "CS3|CS2"
- board text removed: "D0|A0"
- board text removed: "D1|A1"
- board text removed: "D3|A3"
- board text removed: "EN|DRV_GP"
- board text removed: "GND|GND"
- board text removed: "MISO|MOSI"
- board text removed: "PWM1|A"
- board text removed: "PWM2|B"
- board text removed: "PWM3|Z"
- board text removed: "PWM4|GND"
- board text removed: "SCK|CS1"
- board text removed: "V_INT|V_EXT"
